Commit message: Replace coarse link meshes with SO-101 parts and bring pick-and-place, the pendant, and pose registration in line with that arm.
Co-authored-by: Cursor <cursoragent@cursor.com>

File: pendant/SO101_6DOF.urdf (robot description, URDF)
Before this commit: robot SO101_6DOF, 8 links, 7 joints
Links:
- link BASE_1: mass 1.4138178700759005 -> 0.147; geometry collision mesh filename=package://meshes/base_motor_holder_so101_v1.stl; collision mesh filename=package://meshes/base_so101_v2.stl
- link L1_1: mass 0.9302287393788501 -> 0.100006; geometry collision mesh filename=package://meshes/motor_holder_so101_base_v1.stl; collision mesh filename=package://meshes/rotation_pitch_so101_v1.stl
- link L2_1: mass 1.2731856908289911 -> 0.103; geometry collision mesh filename=package://meshes/sts3215_03a_v1.stl; collision mesh filename=package://meshes/upper_arm_so101_v1.stl
- link L3_1: mass 0.5075940741079121 -> 0.104; geometry collision mesh filename=package://meshes/sts3215_03a_no_horn_v1.stl; collision mesh filename=package://meshes/wrist_roll_pitch_so101_v2.stl
- link L4_1: mass 0.6716678130372074 -> 0.04
- link L5_1: mass 0.5075938722215222 -> 0.079; geometry collision mesh filename=package://meshes/sts3215_03a_no_horn_v1.stl; collision mesh filename=package://meshes/wrist_roll_pitch_so101_v2.stl
- link L6_1: mass 0.6955792923870261 -> 0.087; geometry collision mesh filename=package://meshes/sts3215_03a_v1.stl; collision mesh filename=package://meshes/wrist_roll_follower_so101_v1.stl
- link L7_1: mass 0.1586832108582172 -> 0.012; geometry collision mesh filename=package://meshes/moving_jaw_so101_v1.stl; visual mesh filename=package://meshes/moving_jaw_so101_v1.stl
Joints:
- joint S1: axis 0.0 0.0 1.0 -> 0 0 1; limit lower=-3.14159 upper=3.14159 effort=100 velocity=100 -> lower=-1.91986 upper=1.91986 effort=10 velocity=10; origin xyz=1.0269904119381793e-05 -0.006491919613632658 0.06469999999999797 rpy=0 0 0 -> xyz=0 0 0.0624 rpy=3.14159 4.18253e-17 -3.14159
- joint S2: axis 1.0 3.899658373995775e-15 9.973680369662098e-15 -> 0 0 1; limit lower=-3.14159 upper=3.14159 effort=100 velocity=100 -> lower=-1.74533 upper=1.74533 effort=10 velocity=10; origin xyz=0.017932829246147305 -0.030485842405230848 0.054101779329775 rpy=0 0 0 -> xyz=-0.0303992 -0.0182778 -0.0542 rpy=-1.5708 -1.5708 0
- joint S3: axis 1.0 4.315992008230064e-15 1.3031262354691917e-14 -> 0 0 1; limit lower=-3.14159 upper=3.14159 effort=100 velocity=100 -> lower=-1.69 upper=1.69 effort=10 velocity=10; origin xyz=0.0004378052362622488 -0.11290778347202711 -0.02800000000000151 rpy=0 0 0 -> xyz=-0.11257 -0.028 0 rpy=0 0 0
- joint S4: axis 6.661013685071851e-10 -1.0 -8.495972595381182e-16 -> 0 1 0; limit lower=-3.14159 upper=3.14159 effort=100 velocity=100 -> lower=-3.14159 upper=3.14159 effort=10 velocity=10; origin xyz=-0.017999999961253677 -0.0598672286542527 0.00113277134574985 rpy=0 0 0 -> xyz=0 -0.0611 0.0181 rpy=0 0 0
- joint S5: axis -1.0 -1.333394269997649e-09 -6.661193142758406e-10 -> 0 0 -1; limit lower=-3.14159 upper=3.14159 effort=100 velocity=100 -> lower=-1.65806 upper=1.65806 effort=10 velocity=10; origin xyz=-0.01820545145418451 -0.07311480043157165 -0.004986129102844447 rpy=0 0 0 -> xyz=0.004986129102844447 -0.07311480043157165 -0.01820545145418451 rpy=0 0 0
- joint S6: axis 6.666111507521254e-10 -0.9999999906839232 0.0001364996476153662 -> 0 0 1; limit lower=-3.14159 upper=3.14159 effort=100 velocity=100 -> lower=-2.74385 upper=2.84121 effort=10 velocity=10; origin xyz=0.018000000041797887 -0.05986738269542291 -0.0011245994675887494 rpy=0 0 0 -> xyz=5.55112e-17 -0.0611 0.0181 rpy=1.5708 0.0486795 3.14159
- joint S7: axis 1.6654672358491272e-09 -0.00013649965749629398 -0.9999999906839215 -> 0 0 1; limit lower=-3.14159 upper=3.14159 effort=100 velocity=100 -> lower=-0.174533 upper=1.74533 effort=10 velocity=10; origin xyz=0.02020000003980696 -0.02503979464791689 -0.016809082194564645 rpy=0 0 0 -> xyz=0.0202 0.0188 -0.0234 rpy=1.5708 -5.24284e-08 -1.41553e-15
